File: cad_files/mini-serial-console.kicad_pcb (KiCad board)
At the start: 2 copper layers, 97.8 x 59.7 mm, 8 parts

Commit message: 220929
Parts:
- removed the REF** at (117.5, 105.4)
- added C1: 1000u, Capacitors_THT:CP_Radial_D10.0mm_P5.00mm, F.Cu at (146.1, 101.6)
- added C2: 100n, Capacitors_THT:C_Disc_D5.0mm_W2.5mm_P5.00mm, F.Cu at (69.8, 100.3)
- added C3: 100n, Capacitors_THT:C_Disc_D5.0mm_W2.5mm_P5.00mm, F.Cu at (67.3, 57.1)
- added C4: 100n, Capacitors_THT:C_Disc_D5.0mm_W2.5mm_P5.00mm, F.Cu at (135.9, 97.8)
- added C5: 100n, Capacitors_THT:C_Disc_D5.0mm_W2.5mm_P5.00mm, F.Cu at (134.6, 78.7)
- added D1: 1N4001, Diodes_THT:D_DO-41_SOD81_P10.16mm_Horizontal, F.Cu at (130.8, 86.4)
- added D2: 1N4148, Diodes_THT:D_DO-41_SOD81_P7.62mm_Horizontal, F.Cu at (124.5, 87.6)
- added F1: Fuse, Fuse_holders:Fuseholder5x20_simple_metal, F.Cu at (138.4, 92.7)
- added J1: Screw_Terminal_1x02, Connectors:bornier2, F.Cu at (158.8, 92.7)
- added J2: Screw_Terminal_1x03, Connectors:bornier3, F.Cu at (125.7, 52.1)
- added J4: Screw_Terminal_1x05, Connectors:bornier5, F.Cu at (139.7, 104.1)
- added JP1: Jumper_NO_Small, Socket_Strips:Socket_Strip_Straight_1x02, F.Cu at (124.5, 66.0)
- added JP2: Jumper_NO_Small, Socket_Strips:Socket_Strip_Straight_1x02, F.Cu at (124.5, 73.7)
- added JP3: Jumper_NC_Small, Socket_Strips:Socket_Strip_Straight_1x02, F.Cu at (124.5, 62.2)
- added JP4: Jumper_NC_Small, Socket_Strips:Socket_Strip_Straight_1x02, F.Cu at (124.5, 69.8)
- added JP5: Jumper_NO_Small, Socket_Strips:Socket_Strip_Straight_1x02, F.Cu at (91.4, 54.6)
- added JP6: Jumper_NO_Small, Socket_Strips:Socket_Strip_Straight_1x02, F.Cu at (111.8, 52.1)
- added JP7: Jumper_NO_Small, Socket_Strips:Socket_Strip_Straight_1x02, F.Cu at (115.6, 52.1)
- added P1: 10k, Potentiometers:Potentiometer_WirePads_Small, F.Cu at (69.8, 92.1)
- added Q1: BC559, TO_SOT_Packages_THT:TO-92_Inline_Narrow_Oval, F.Cu at (139.7, 77.5)
- added Q2: BC548, TO_SOT_Packages_THT:TO-92_Inline_Narrow_Oval, F.Cu at (129.5, 77.5)
- added R1: 560, Resistors_THT:R_Axial_DIN0411_L9.9mm_D3.6mm_P12.70mm_Horizontal, F.Cu at (106.7, 87.6)
- added R10: 10k, Resistors_THT:R_Axial_DIN0411_L9.9mm_D3.6mm_P12.70mm_Horizontal, F.Cu at (83.8, 92.1)
- added R11: 10k, Resistors_THT:R_Axial_DIN0411_L9.9mm_D3.6mm_P12.70mm_Horizontal, F.Cu at (108.0, 52.1)
- added R12: 10k, Resistors_THT:R_Axial_DIN0411_L9.9mm_D3.6mm_P12.70mm_Horizontal, F.Cu at (83.8, 87.6)
- added R13: 10k, Resistors_THT:R_Axial_DIN0411_L9.9mm_D3.6mm_P12.70mm_Horizontal, F.Cu at (108.0, 55.9)
- added R2: 10k, Resistors_THT:R_Axial_DIN0411_L9.9mm_D3.6mm_P12.70mm_Horizontal, F.Cu at (111.8, 100.3)
- added R3: 10k, Resistors_THT:R_Axial_DIN0411_L9.9mm_D3.6mm_P12.70mm_Horizontal, F.Cu at (120.7, 92.7)
- added R4: 10k, Resistors_THT:R_Axial_DIN0411_L9.9mm_D3.6mm_P12.70mm_Horizontal, F.Cu at (134.6, 58.4)
- added R5: 4.7k, Resistors_THT:R_Axial_DIN0411_L9.9mm_D3.6mm_P12.70mm_Horizontal, F.Cu at (141.0, 82.5)
- added R6: 4.7k, Resistors_THT:R_Axial_DIN0411_L9.9mm_D3.6mm_P12.70mm_Horizontal, F.Cu at (139.7, 58.4)
- added R7: 10k, Resistors_THT:R_Axial_DIN0411_L9.9mm_D3.6mm_P12.70mm_Horizontal, F.Cu at (83.8, 101.0)
- added R8: 10k, Resistors_THT:R_Axial_DIN0411_L9.9mm_D3.6mm_P12.70mm_Horizontal, F.Cu at (83.8, 96.5)
- added R9: 4.7k, Resistors_THT:R_Axial_DIN0411_L9.9mm_D3.6mm_P12.70mm_Horizontal, F.Cu at (129.5, 71.1)
- J3: renamed from REF**; value DB9MC -> DB9M
- U1: renamed from REF**; value Socket_Strip_Straight_1x16 -> HD44780 compatible LCD
- U2: renamed from REF**; value RPi_Pico_SMD_TH -> Pico
- moved U2 5.72 mm to (91.4, 72.4)
Connections:
- J3 pad 1: (no net) -> Net-(J3-Pad1)
- J3 pad 2: (no net) -> /TXD-RS232C
- J3 pad 3: (no net) -> /RXD-RS232C
- J3 pad 4: (no net) -> Net-(J3-Pad4)
- J3 pad 5: (no net) -> GND
- J3 pad 6: (no net) -> Net-(J3-Pad6)
- J3 pad 7: (no net) -> Net-(J3-Pad7)
- J3 pad 8: (no net) -> Net-(J3-Pad8)
- J3 pad 9: (no net) -> Net-(J3-Pad9)
- U1 pad 1: (no net) -> +5V
- U1 pad 10: (no net) -> /DB3
- U1 pad 11: (no net) -> /DB4
- U1 pad 12: (no net) -> /DB5
- U1 pad 13: (no net) -> /DB6
- U1 pad 14: (no net) -> /DB7
- U1 pad 15: (no net) -> /BL+
- U1 pad 16: (no net) -> GND
- U1 pad 2: (no net) -> GND
- U1 pad 3: (no net) -> /CONT
- U1 pad 4: (no net) -> /RS
- U1 pad 5: (no net) -> GND
- U1 pad 6: (no net) -> /EN
- U1 pad 7: (no net) -> /DB0
- U1 pad 8: (no net) -> /DB1
- U1 pad 9: (no net) -> /DB2
- U2 pad 1: (no net) -> /TXD
- U2 pad 10: (no net) -> /DB5
- U2 pad 11: (no net) -> /DB6
- U2 pad 12: (no net) -> /DB7
- U2 pad 13: (no net) -> Net-(U2-Pad13)
- U2 pad 14: (no net) -> /EN
- U2 pad 15: (no net) -> /RS
- U2 pad 16: (no net) -> /-BU
- U2 pad 17: (no net) -> /-BD
- U2 pad 18: (no net) -> /BC
- U2 pad 19: (no net) -> /-BL
- U2 pad 2: (no net) -> /RXD
- U2 pad 20: (no net) -> /-BR
- U2 pad 21: (no net) -> /-LB
- U2 pad 22: (no net) -> /-AS
- U2 pad 23: (no net) -> /JC
- U2 pad 24: (no net) -> Net-(U2-Pad24)
- U2 pad 25: (no net) -> Net-(U2-Pad25)
- U2 pad 26: (no net) -> Net-(U2-Pad26)
- U2 pad 27: (no net) -> Net-(U2-Pad27)
- U2 pad 28: (no net) -> Net-(U2-Pad28)
- U2 pad 29: (no net) -> Net-(U2-Pad29)
- U2 pad 3: (no net) -> Net-(U2-Pad3)
- U2 pad 30: (no net) -> /-RST
- U2 pad 31: (no net) -> Net-(U2-Pad31)
- U2 pad 32: (no net) -> Net-(U2-Pad32)
- U2 pad 33: (no net) -> GND
- U2 pad 34: (no net) -> Net-(U2-Pad34)
- U2 pad 35: (no net) -> Net-(U2-Pad35)
- U2 pad 36: (no net) -> Net-(U2-Pad36)
- U2 pad 37: (no net) -> Net-(U2-Pad37)
- U2 pad 38: (no net) -> GND
- U2 pad 39: (no net) -> Net-(U2-Pad39)
- U2 pad 4: (no net) -> /DB0
- U2 pad 40: (no net) -> +5V
- U2 pad 41: (no net) -> Net-(U2-Pad41)
- U2 pad 42: (no net) -> Net-(U2-Pad42)
- U2 pad 43: (no net) -> Net-(U2-Pad43)
- U2 pad 5: (no net) -> /DB1
- U2 pad 6: (no net) -> /DB2
- U2 pad 7: (no net) -> /DB3
- U2 pad 8: (no net) -> Net-(U2-Pad8)
- U2 pad 9: (no net) -> /DB4
Routing:
- net /-LB: track 0.00 -> 18.8 mm
- net /JC: track 0.00 -> 17.0 mm
- net /-AS: track 0.00 -> 14.3 mm
- net /-RST: track 0.00 -> 9.42 mm
- net +5V: track 0.00 -> 3.81 mm
- net /-BL: track 0.00 -> 2.54 mm

Commit message: 220930
Parts:
- removed JP4: Jumper_NC_Small, Socket_Strips:Socket_Strip_Straight_1x02
- removed JP5, JP6, JP7: Jumper_NO_Small, Socket_Strips:Socket_Strip_Straight_1x02
- removed P1: 10k, Potentiometers:Potentiometer_WirePads_Small
- added Q3: BC548, TO_SOT_Packages_THT:TO-92_Inline_Narrow_Oval, F.Cu at (186.7, 146.1)
- added R14: 4.7k, Resistors_THT:R_Axial_DIN0411_L9.9mm_D3.6mm_P12.70mm_Horizontal, F.Cu at (165.1, 134.6)
- added R15: 4.7k, Resistors_THT:R_Axial_DIN0411_L9.9mm_D3.6mm_P12.70mm_Horizontal, F.Cu at (165.1, 141.0)
- J3: value DB9M -> Screw_Terminal_1x03; footprint Connectors:DB9MC -> Connectors:bornier3
- JP3: value Jumper_NC_Small -> Jumper_NO_Small
- Q1: value BC559 -> BC109; footprint TO_SOT_Packages_THT:TO-92_Inline_Narrow_Oval -> TO_SOT_Packages_THT:TO-18-3
- Q2: value BC548 -> BC559
- R3: value 10k -> 1k
- R5, R6, R9: value 4.7k -> 10k
- R7: value 10k -> 4.7k
- moved R11 97.2 mm to (147.3, 141.0), turned to 0 degrees
- moved C5 92.5 mm to (200.7, 143.5), turned to 180 degrees
- moved R13 92.2 mm to (165.1, 128.3), turned to 0 degrees
- moved R4 91.8 mm to (111.8, 147.3), turned to 0 degrees
- moved R12 87.2 mm to (147.3, 147.3)
- moved D2 84.3 mm to (196.8, 130.8), turned to 0 degrees
- moved Q2 82.6 mm to (186.7, 137.2), turned to 0 degrees
- moved D1 77.5 mm to (196.8, 127.0)
- moved R6 76.9 mm to (129.5, 134.6), turned to 0 degrees
- moved JP3 76.8 mm to (102.9, 135.9)
- moved R10 76.4 mm to (147.3, 134.6)
- moved C1 75.2 mm to (215.9, 129.5)
- moved C4 72.9 mm to (195.6, 139.7)
- moved J2 72.4 mm to (195.6, 71.1), turned to 270 degrees
- moved Q1 70.1 mm to (186.7, 129.5), turned to 0 degrees
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Connections:
- J3 pad 1: Net-(J3-Pad1) -> /TXD-RS232C
- J3 pad 2: /TXD-RS232C -> /RXD-RS232C
- J3 pad 3: /RXD-RS232C -> GND
- J4 pad 1: /BC -> GND
- J4 pad 2: /-BR -> Net-(J4-Pad2)
- J4 pad 3: /-BL -> Net-(J4-Pad3)
- J4 pad 4: /-BD -> Net-(J4-Pad4)
- J4 pad 5: /-BU -> Net-(J4-Pad5)
- JP1 pad 1: /TXD-TTL -> Net-(JP1-Pad1)
- JP1 pad 2: /TXD -> GND
- JP2 pad 1: /RXD-TTL -> Net-(JP2-Pad1)
- JP2 pad 2: /RXD -> GND
- JP3 pad 2: /TXD -> GND
- Q1 pad 1: +5V -> Net-(Q1-Pad1)
- Q1 pad 3: /TXD-RS232C -> GND
- Q2 pad 1: Net-(JP4-Pad1) -> +5V
- Q2 pad 3: GND -> /TXD-RS232C
- R1 pad 1: +5V -> Net-(R1-Pad1)
- R1 pad 2: /BL+ -> Net-(Q1-Pad1)
- R10 pad 2: /-BL -> Net-(J4-Pad3)
- R11 pad 1: /-AS -> +5V
- R11 pad 2: +5V -> Net-(J4-Pad2)
- R12 pad 2: /-BR -> Net-(JP2-Pad1)
- R13 pad 1: /-LB -> +5V
- R13 pad 2: +5V -> Net-(JP3-Pad1)
- R2 pad 1: +5V -> Net-(R2-Pad1)
- R2 pad 2: Net-(Q1-Pad2) -> GND
- R3 pad 1: +5V -> Net-(Q1-Pad2)
- R3 pad 2: Net-(JP4-Pad1) -> /BL
- R4 pad 1: Net-(JP3-Pad1) -> +5V
- R4 pad 2: Net-(Q1-Pad2) -> Net-(Q2-Pad2)
- R5 pad 1: /TXD-RS232C -> +5V
- R5 pad 2: Net-(C5-Pad1) -> /RXD1
- R6 pad 1: Net-(Q2-Pad2) -> /TXD1
- R6 pad 2: /RXD-RS232C -> Net-(Q2-Pad2)
- R7 pad 1: +5V -> /TXD-RS232C
- R7 pad 2: /-BU -> Net-(C5-Pad1)
- R8 pad 2: /-BD -> Net-(J4-Pad4)
- R9 pad 1: Net-(Q2-Pad2) -> +5V
- R9 pad 2: GND -> Net-(J4-Pad5)
- U1 pad 15: /BL+ -> +5V
- U1 pad 16: GND -> Net-(R1-Pad1)
- U1 pad 3: /CONT -> Net-(R2-Pad1)
- U2 pad 1: /TXD -> /TXD-TTL
- U2 pad 10: /DB5 -> Net-(U2-Pad10)
- U2 pad 11: /DB6 -> /TXD1
- U2 pad 12: /DB7 -> /RXD1
- U2 pad 13: Net-(U2-Pad13) -> GND
- U2 pad 14: /EN -> /DB4
- U2 pad 15: /RS -> /DB5
- U2 pad 16: /-BU -> /DB6
- U2 pad 17: /-BD -> /DB7
- U2 pad 18: /BC -> GND
- U2 pad 19: /-BL -> /EN
- U2 pad 2: /RXD -> /RXD-TTL
- U2 pad 20: /-BR -> /RS
- U2 pad 21: /-LB -> Net-(JP3-Pad1)
- U2 pad 22: /-AS -> Net-(JP2-Pad1)
- U2 pad 23: /JC -> GND
- U2 pad 24: Net-(U2-Pad24) -> Net-(J4-Pad2)
- U2 pad 25: Net-(U2-Pad25) -> Net-(J4-Pad3)
- U2 pad 26: Net-(U2-Pad26) -> Net-(J4-Pad4)
- U2 pad 27: Net-(U2-Pad27) -> Net-(J4-Pad5)
- U2 pad 28: Net-(U2-Pad28) -> GND
- U2 pad 3: Net-(U2-Pad3) -> GND
- U2 pad 30: /-RST -> Net-(JP1-Pad1)
- U2 pad 42: Net-(U2-Pad42) -> GND
- U2 pad 8: Net-(U2-Pad8) -> GND
- U2 pad 9: /DB4 -> /BL
Routing:
- net /-LB: track 18.8 -> 0.00 mm
- net /JC: track 17.0 -> 0.00 mm
- net /-AS: track 14.3 -> 0.00 mm
- net /-RST: track 9.42 -> 0.00 mm
- net +5V: track 3.81 -> 0.00 mm
- net (no net): track 0.00 -> 3.81 mm
- net /EN: track 0.00 -> 2.54 mm
- net /-BL: track 2.54 -> 0.00 mm

Commit message: 220930
Parts:
- added R16: 1k, Resistors_THT:R_Axial_DIN0309_L9.0mm_D3.2mm_P5.08mm_Vertical, F.Cu at (147.3, 128.3)
- added R17: 1k, Resistors_THT:R_Axial_DIN0309_L9.0mm_D3.2mm_P5.08mm_Vertical, F.Cu at (147.3, 134.6)
- added R18: 10k, Resistors_THT:R_Axial_DIN0309_L9.0mm_D3.2mm_P5.08mm_Vertical, F.Cu at (147.3, 141.0)
- added R19: 10k, Resistors_THT:R_Axial_DIN0309_L9.0mm_D3.2mm_P5.08mm_Vertical, F.Cu at (147.3, 147.3)
- added R20: 10k, Resistors_THT:R_Axial_DIN0309_L9.0mm_D3.2mm_P5.08mm_Vertical, F.Cu at (147.3, 153.7)
- added R21: 10k, Resistors_THT:R_Axial_DIN0309_L9.0mm_D3.2mm_P5.08mm_Vertical, F.Cu at (158.8, 128.3)
- added R22: 10k, Resistors_THT:R_Axial_DIN0309_L9.0mm_D3.2mm_P5.08mm_Vertical, F.Cu at (158.8, 134.6)
- added R23: 10k, Resistors_THT:R_Axial_DIN0309_L9.0mm_D3.2mm_P5.08mm_Vertical, F.Cu at (158.8, 141.0)
- added R24: 10k, Resistors_THT:R_Axial_DIN0309_L9.0mm_D3.2mm_P5.08mm_Vertical, F.Cu at (158.8, 147.3)
- added R25: 10k, Resistors_THT:R_Axial_DIN0309_L9.0mm_D3.2mm_P5.08mm_Vertical, F.Cu at (158.8, 153.7)
- F1: value Fuse -> 1A F
- J4: value Screw_Terminal_1x05 -> Screw_Terminal_1x07; footprint Connectors:bornier5 -> Bornier:bornier7
- Q1: value BC109 -> BC559; footprint TO_SOT_Packages_THT:TO-18-3 -> TO_SOT_Packages_THT:TO-92_Inline_Narrow_Oval
- Q2: value BC559 -> BC548
- Q3: value BC548 -> BC109; footprint TO_SOT_Packages_THT:TO-92_Inline_Narrow_Oval -> TO_SOT_Packages_THT:TO-18-3
- R1: value 560 -> 4.7k; footprint Resistors_THT:R_Axial_DIN0411_L9.9mm_D3.6mm_P12.70mm_Horizontal -> Resistors_THT:R_Axial_DIN0309_L9.0mm_D3.2mm_P5.08mm_Vertical
- R10, R11, R12, R13, R9: value 10k -> 1k; footprint Resistors_THT:R_Axial_DIN0411_L9.9mm_D3.6mm_P12.70mm_Horizontal -> Resistors_THT:R_Axial_DIN0309_L9.0mm_D3.2mm_P5.08mm_Vertical
- R14, R15: value 4.7k -> 1k; footprint Resistors_THT:R_Axial_DIN0411_L9.9mm_D3.6mm_P12.70mm_Horizontal -> Resistors_THT:R_Axial_DIN0309_L9.0mm_D3.2mm_P5.08mm_Vertical
- R2, R4: value 10k -> 4.7k; footprint Resistors_THT:R_Axial_DIN0411_L9.9mm_D3.6mm_P12.70mm_Horizontal -> Resistors_THT:R_Axial_DIN0309_L9.0mm_D3.2mm_P5.08mm_Vertical
- R3: value 1k -> 10k; footprint Resistors_THT:R_Axial_DIN0411_L9.9mm_D3.6mm_P12.70mm_Horizontal -> Resistors_THT:R_Axial_DIN0309_L9.0mm_D3.2mm_P5.08mm_Vertical
- R5, R6: footprint Resistors_THT:R_Axial_DIN0411_L9.9mm_D3.6mm_P12.70mm_Horizontal -> Resistors_THT:R_Axial_DIN0309_L9.0mm_D3.2mm_P5.08mm_Vertical
- R7: value 4.7k -> 10k; footprint Resistors_THT:R_Axial_DIN0411_L9.9mm_D3.6mm_P12.70mm_Horizontal -> Resistors_THT:R_Axial_DIN0309_L9.0mm_D3.2mm_P5.08mm_Vertical
- R8: value 10k -> 560; footprint Resistors_THT:R_Axial_DIN0411_L9.9mm_D3.6mm_P12.70mm_Horizontal -> Resistors_THT:R_Axial_DIN0309_L9.0mm_D3.2mm_P5.08mm_Vertical
- U2: value Pico -> Raspberry Pi Pico
- moved C1 41.6 mm to (180.3, 151.1)
- moved R13 31.9 mm to (135.9, 141.0)
- moved R14 31.9 mm to (135.9, 147.3)
- moved R15 31.9 mm to (135.9, 153.7)
- moved R5 30.3 mm to (113.0, 153.7)
- moved R10 29.8 mm to (124.5, 153.7)
- moved R9 29.8 mm to (124.5, 147.3)
- moved D1 17.8 mm to (179.1, 127.0)
- moved D2 17.8 mm to (179.1, 130.8)
- moved R11 17.1 mm to (135.9, 128.3)
- moved R12 17.1 mm to (135.9, 134.6)
- moved C4 16.7 mm to (179.1, 137.2)
- moved C5 16.7 mm to (184.2, 141.0)
- moved Q1 16.6 mm to (170.2, 128.3)
- moved Q2 16.5 mm to (170.2, 137.2)
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Connections:
- net /RXD-TTL renamed /RXD0
- net /TXD-TTL renamed /TXD0
- C3 pad 1: +5V -> Net-(C3-Pad1)
- C5 pad 1: Net-(C5-Pad1) -> +5V
- D2 pad 1: /RXD-RS232C -> /RXD1-RS232C
- D2 pad 2: Net-(C5-Pad1) -> Net-(C3-Pad1)
- J3 pad 1: /TXD-RS232C -> /TXD1-RS232C
- J3 pad 2: /RXD-RS232C -> /RXD1-RS232C
- J4 pad 2: Net-(J4-Pad2) -> /PB0
- J4 pad 3: Net-(J4-Pad3) -> /PB1
- J4 pad 4: Net-(J4-Pad4) -> /PB2
- J4 pad 5: Net-(J4-Pad5) -> /PB3
- JP2 pad 1: Net-(JP2-Pad1) -> GND
- JP2 pad 2: GND -> Net-(JP2-Pad2)
- JP3 pad 1: Net-(JP3-Pad1) -> GND
- JP3 pad 2: GND -> Net-(JP3-Pad2)
- Q1 pad 1: Net-(Q1-Pad1) -> +5V
- Q1 pad 3: GND -> /TXD1-RS232C
- Q2 pad 1: +5V -> /RXD1
- Q2 pad 3: /TXD-RS232C -> GND
- Q3 pad 1: /RXD1 -> Net-(Q3-Pad1)
- R1 pad 1: Net-(R1-Pad1) -> /TXD1-RS232C
- R1 pad 2: Net-(Q1-Pad1) -> Net-(C3-Pad1)
- R10 pad 1: +5V -> /PB4
- R10 pad 2: Net-(J4-Pad3) -> Net-(R10-Pad2)
- R11 pad 1: +5V -> /PB3
- R11 pad 2: Net-(J4-Pad2) -> Net-(R11-Pad2)
- R12 pad 1: +5V -> /PB2
- R12 pad 2: Net-(JP2-Pad1) -> Net-(R12-Pad2)
- R13 pad 1: +5V -> /PB1
- R13 pad 2: Net-(JP3-Pad1) -> Net-(R13-Pad2)
- R14 pad 1: Net-(Q3-Pad2) -> /PB0
- R14 pad 2: /RXD-RS232C -> Net-(R14-Pad2)
- R15 pad 1: Net-(Q3-Pad2) -> Net-(JP2-Pad2)
- R15 pad 2: GND -> Net-(R15-Pad2)
- R2 pad 1: Net-(R2-Pad1) -> Net-(Q2-Pad2)
- R2 pad 2: GND -> /RXD1-RS232C
- R3 pad 1: Net-(Q1-Pad2) -> +5V
- R3 pad 2: /BL -> Net-(Q1-Pad2)
- R4 pad 1: +5V -> Net-(Q2-Pad2)
- R4 pad 2: Net-(Q2-Pad2) -> GND
- R5 pad 1: +5V -> /TXD1
- R5 pad 2: /RXD1 -> Net-(Q1-Pad2)
- R6 pad 1: /TXD1 -> +5V
- R6 pad 2: Net-(Q2-Pad2) -> /RXD1
- R7 pad 1: /TXD-RS232C -> Net-(R7-Pad1)
- R7 pad 2: Net-(C5-Pad1) -> GND
- R8 pad 1: +5V -> Net-(R8-Pad1)
- R8 pad 2: Net-(J4-Pad4) -> Net-(Q3-Pad1)
- R9 pad 1: +5V -> /PB5
- R9 pad 2: Net-(J4-Pad5) -> Net-(R9-Pad2)
- U1 pad 16: Net-(R1-Pad1) -> Net-(R8-Pad1)
- U1 pad 3: Net-(R2-Pad1) -> Net-(R7-Pad1)
- U2 pad 10: Net-(U2-Pad10) -> /EN
- U2 pad 19: /EN -> /BL
- U2 pad 20: /RS -> Net-(R16-Pad2)
- U2 pad 21: Net-(JP3-Pad1) -> Net-(R15-Pad2)
- U2 pad 22: Net-(JP2-Pad1) -> Net-(R14-Pad2)
- U2 pad 24: Net-(J4-Pad2) -> Net-(R13-Pad2)
- U2 pad 25: Net-(J4-Pad3) -> Net-(R12-Pad2)
- U2 pad 26: Net-(J4-Pad4) -> Net-(R11-Pad2)
- U2 pad 27: Net-(J4-Pad5) -> Net-(R10-Pad2)
- U2 pad 29: Net-(U2-Pad29) -> Net-(R9-Pad2)
- U2 pad 9: /BL -> /RS
Routing:
- net /EN: track 2.54 -> 0.00 mm
- net (no net): track 3.81 -> 2.54 mm

Commit message: 221001
Parts:
- moved R3 97.1 mm to (185.4, 76.2), turned to 270 degrees
- moved C4 95.0 mm to (104.1, 78.7)
- moved R20 90.1 mm to (137.2, 64.1), turned to 270 degrees
- moved R19 84.3 mm to (133.3, 64.1), turned to 270 degrees
- moved R1 84.1 mm to (179.1, 76.2), turned to 270 degrees
- moved R10 79.9 mm to (133.3, 74.3), turned to 270 degrees
- moved R4 79.6 mm to (167.1, 88.9), turned to 270 degrees
- moved R18 78.9 mm to (129.5, 64.1), turned to 270 degrees
- moved R2 77.5 mm to (179.1, 94.0), turned to 90 degrees
- moved R23 77.3 mm to (149.9, 64.1), turned to 270 degrees
- moved R14 74.3 mm to (149.9, 74.3), turned to 270 degrees
- moved R9 73.2 mm to (129.5, 74.3), turned to 270 degrees
- moved R22 71.9 mm to (144.8, 64.1), turned to 270 degrees
- moved C3 70.5 mm to (172.7, 88.9), turned to 270 degrees
- moved R13 67.3 mm to (144.8, 74.3), turned to 270 degrees
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Routing:
- net GND: track 0.00 -> 485.0 mm
- net +5V: track 0.00 -> 393.8 mm
- net /TXD0: track 0.00 -> 119.8 mm, vias 0 -> 3
- net /RXD0: track 0.00 -> 117.5 mm, vias 0 -> 3
- net Net-(Q1-Pad2): track 0.00 -> 84.9 mm, vias 0 -> 1
- net /PB5: track 0.00 -> 80.4 mm, vias 0 -> 1
- net /PB4: track 0.00 -> 70.3 mm, vias 0 -> 1
- net /PB3: track 0.00 -> 60.1 mm, vias 0 -> 1
- net Net-(JP1-Pad1): track 0.00 -> 50.6 mm, vias 0 -> 2
- net /RXD1: track 0.00 -> 49.5 mm, vias 0 -> 3
- net /PB2: track 0.00 -> 46.5 mm, vias 0 -> 1
- net /TXD1-RS232C: track 0.00 -> 42.3 mm
- net /DB0: track 0.00 -> 41.5 mm, vias 0 -> 2
- net /DB1: track 0.00 -> 38.4 mm, vias 0 -> 2
- net /PB1: track 0.00 -> 37.0 mm, vias 0 -> 1
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Other:
- net class Thick added: clearance 0.2, trace_width 1, via_dia 0.8, via_drill 0.6
- board text added: "* * Mini serial console * *"
- board text added: "2022"
- board text added: "Connectors: J1: +5V DC in J2: TTL serial port J3: RS232C serial port J4: push buttons in"
- board text added: "DN: 59/22/03"
- board text added: "Jumpers: JP1: Reset JP2: Autoscroll JP3: Line break"
- board text added: "http://www.pozsarzs.hu"
