File: cad_files/mini-serial-console.kicad_pcb (KiCad board)
At the start: 2 copper layers, 97.8 x 59.7 mm, 49 parts, among them J1 Screw_Terminal_1x02, J2 Screw_Terminal_1x03, J3 Screw_Terminal_1x03, J4 Screw_Terminal_1x07, Q1 BC559, Q2 BC548, Q3 BC109, U1 HD44780 compatible LCD, U2 Raspberry Pi Pico

Commit message: 221001
Routing:
- net GND: track 485.0 -> 522.2 mm, vias 0 -> 4
Changed lines of the file:
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@@
   (general
     (links 147)
-    (no_connects 3)
+    (no_connects 0)
     (area 96.011429 56.755 204.978572 122.415)
     (thickness 1.6)
     (drawings 19)
-    (tracks 481)
+    (tracks 499)
     (zones 0)
     (modules 49)
@@
     (visible_elements 7FFEF77F)
     (pcbplotparams
-      (layerselection 0x00030_80000001)
+      (layerselection 0x00000_80000000)
       (usegerberextensions false)
-      (excludeedgelayer true)
+      (excludeedgelayer false)
       (linewidth 0.100000)
-      (plotframeref false)
+      (plotframeref true)
       (viasonmask false)
       (mode 1)
@@
       (psa4output false)
       (plotreference true)
-      (plotvalue true)
+      (plotvalue false)
       (plotinvisibletext false)
       (padsonsilk false)
       (subtractmaskfromsilk false)
-      (outputformat 1)
-      (mirror false)
-      (drillshape 0)
+      (outputformat 5)
+      (mirror true)
+      (drillshape 1)
       (scaleselection 1)
       (outputdirectory ""))
@@
   (segment (start 167.64 107.95) (end 167.64 113.665) (width 1) (layer F.Cu) (net 1))
   (segment (start 167.64 113.665) (end 167.005 114.3) (width 1) (layer F.Cu) (net 1))
-  (segment (start 144.78 88.9) (end 146.05 90.17) (width 1) (layer B.Cu) (net 2))
-  (segment (start 146.05 90.17) (end 146.685 90.17) (width 1) (layer B.Cu) (net 2))
+  (via (at 146.304 87.376) (size 0.8) (drill 0.6) (layers F.Cu B.Cu) (net 2))
+  (segment (start 146.304 87.376) (end 146.05 87.376) (width 1) (layer F.Cu) (net 2))
+  (segment (start 147.32 90.805) (end 146.939 90.805) (width 1) (layer B.Cu) (net 2))
+  (segment (start 146.939 90.805) (end 146.304 90.17) (width 1) (layer B.Cu) (net 2))
+  (segment (start 146.05 87.63) (end 146.05 87.376) (width 1) (layer F.Cu) (net 2))
+  (segment (start 147.32 85.09) (end 147.32 86.36) (width 1) (layer F.Cu) (net 2))
+  (segment (start 147.32 86.36) (end 146.05 87.63) (width 1) (layer F.Cu) (net 2))
+  (segment (start 146.05 87.376) (end 146.05 90.17) (width 1) (layer F.Cu) (net 2))
+  (segment (start 147.32 100.965) (end 147.32 102.87) (width 1) (layer F.Cu) (net 2))
+  (segment (start 146.05 99.695) (end 147.32 100.965) (width 1) (layer F.Cu) (net 2))
+  (segment (start 146.05 90.17) (end 146.05 99.695) (width 1) (layer F.Cu) (net 2))
+  (segment (start 146.304 87.376) (end 146.304 90.17) (width 1) (layer B.Cu) (net 2))
+  (segment (start 134.62 85.09) (end 134.62 87.376) (width 1) (layer F.Cu) (net 2))
+  (segment (start 134.62 102.87) (end 134.62 87.376) (width 1) (layer F.Cu) (net 2))
+  (via (at 109.22 87.376) (size 0.8) (drill 0.6) (layers F.Cu B.Cu) (net 2))
+  (segment (start 110.998 87.376) (end 109.22 87.376) (width 1) (layer B.Cu) (net 2))
+  (segment (start 109.22 87.376) (end 109.22 86.36) (width 1) (layer B.Cu) (net 2))
+  (segment (start 109.22 102.87) (end 109.22 87.376) (width 1) (layer F.Cu) (net 2))
+  (segment (start 109.22 87.376) (end 109.22 85.09) (width 1) (layer F.Cu) (net 2))
+  (via (at 121.92 87.376) (size 0.8) (drill 0.6) (layers F.Cu B.Cu) (net 2))
+  (via (at 134.62 87.376) (size 0.8) (drill 0.6) (layers F.Cu B.Cu) (net 2))
+  (segment (start 150.495 93.98) (end 147.32 90.805) (width 1) (layer B.Cu) (net 2))
   (segment (start 152.17 93.98) (end 150.495 93.98) (width 1) (layer B.Cu) (net 2))
-  (segment (start 144.78 88.9) (end 144.78 87.376) (width 1) (layer B.Cu) (net 2))
-  (segment (start 150.495 93.98) (end 146.685 90.17) (width 1) (layer B.Cu) (net 2))
   (segment (start 160.02 91.44) (end 160.02 93.98) (width 1) (layer B.Cu) (net 2) (status 10))
   (segment (start 167.132 93.98) (end 160.528 93.98) (width 1) (layer B.Cu) (net 2))
@@
   (segment (start 121.92 85.09) (end 121.92 87.376) (width 1) (layer B.Cu) (net 2))
   (segment (start 109.22 85.09) (end 109.22 86.36) (width 1) (layer B.Cu) (net 2))
-  (segment (start 109.22 86.36) (end 110.236 87.376) (width 1) (layer B.Cu) (net 2))
-  (segment (start 110.236 87.376) (end 121.92 87.376) (width 1) (layer B.Cu) (net 2))
+  (segment (start 110.998 87.376) (end 121.92 87.376) (width 1) (layer B.Cu) (net 2))
   (segment (start 146.304 87.376) (end 147.32 86.36) (width 1) (layer B.Cu) (net 2))
   (segment (start 144.78 87.376) (end 146.304 87.376) (width 1) (layer B.Cu) (net 2))
   (segment (start 147.32 86.36) (end 147.32 85.09) (width 1) (layer B.Cu) (net 2))
-  (segment (start 121.92 87.376) (end 144.78 87.376) (width 1) (layer B.Cu) (net 2))
-  (segment (start 134.62 102.87) (end 134.62 85.09) (width 1) (layer F.Cu) (net 2))
-  (segment (start 121.92 102.87) (end 121.92 85.09) (width 1) (layer F.Cu) (net 2))
+  (segment (start 121.92 87.376) (end 134.62 87.376) (width 1) (layer B.Cu) (net 2))
+  (segment (start 134.62 87.376) (end 144.78 87.376) (width 1) (layer B.Cu) (net 2))
+  (segment (start 121.92 102.87) (end 121.92 87.376) (width 1) (layer F.Cu) (net 2))
+  (segment (start 121.92 87.376) (end 121.92 85.09) (width 1) (layer F.Cu) (net 2))
   (segment (start 121.92 109.22) (end 121.92 102.87) (width 1) (layer F.Cu) (net 2))
   (segment (start 109.855 107.95) (end 102.235 107.95) (width 1) (layer B.Cu) (net 2) (status 10))

Commit message: 221009
Parts:
- moved C2 4.95 mm to (114.8, 111.8), turned to 180 degrees
Connections:
- U1 pad 1: +5V -> GND
- U1 pad 2: GND -> +5V
Routing:
- net GND: track 522.2 -> 524.4 mm

Commit message: 221018
Parts:
- moved REF** 117.2 mm to (98.6, 126.0), turned to 180 degrees
- moved REF** 108.3 mm to (98.6, 71.4), turned to 180 degrees
- moved REF** 108.0 mm to (191.3, 126.0), turned to 180 degrees
- moved J2 106.2 mm to (99.8, 117.1), turned to 90 degrees
- moved REF** 98.3 mm to (191.3, 71.4), turned to 180 degrees
- moved J1 97.8 mm to (99.8, 84.1), turned to 90 degrees
- moved J3 96.6 mm to (99.8, 100.6), turned to 90 degrees
- moved C4 92.4 mm to (191.3, 109.5), turned to 180 degrees
- moved U1 86.1 mm to (184.3, 71.4), turned to 180 degrees
- moved R3 83.5 mm to (110.0, 112.0), turned to 90 degrees
- moved D2 80.0 mm to (108.7, 103.1), turned to 0 degrees
- moved Q1 78.0 mm to (108.7, 94.2), turned to 270 degrees
- moved C1 76.9 mm to (110.0, 86.6), turned to 90 degrees
- moved C2 74.7 mm to (180.6, 76.5), turned to 0 degrees
- moved F1 72.5 mm to (117.6, 73.9), turned to 180 degrees
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Connections:
- JP1 pad 1: Net-(JP1-Pad1) -> GND
- JP1 pad 2: GND -> Net-(JP1-Pad2)
- U2 pad 30: Net-(JP1-Pad1) -> Net-(JP1-Pad2)
Routing:
- net Net-(JP1-Pad1): track 50.6 -> 0.00 mm, vias 2 -> 0
- net Net-(JP1-Pad2): track 0.00 -> 50.6 mm, vias 0 -> 2
Other:
- board text added: "JP3 JP2 #1 O O #2 O C #3 C O #4 C C"
- board text added: "Op. mode"
- board text added: "Operation modes:"
- board text added: "Reset"
- board text removed: "Jumpers: JP1: Reset JP2: Autoscroll JP3: Line break"
