File: cad_files/mini-serial-console.sch (KiCad schematic (older format))
At the start: 37 parts, among them J1 Screw_Terminal_1x02, J2 Screw_Terminal_1x03, J3 DB9M, J4 Screw_Terminal_1x05, P1 10k, Q1 BC559, Q2 BC548, U1 HD44780 compatible LCD, U2 Pico

Commit message: 220929
Parts:
- C1: footprint (none) -> Capacitors_THT:CP_Radial_D10.0mm_P5.00mm
- C2, C3, C4, C5: footprint (none) -> Capacitors_THT:C_Disc_D5.0mm_W2.5mm_P5.00mm
- D1: footprint (none) -> Diodes_THT:D_DO-41_SOD81_P10.16mm_Horizontal
- D2: footprint (none) -> Diodes_THT:D_DO-41_SOD81_P7.62mm_Horizontal
- F1: footprint (none) -> Fuse_holders:Fuseholder5x20_simple_metal
- J1: footprint (none) -> Connectors:bornier2
- J2: footprint (none) -> Connectors:bornier3
- J4: footprint (none) -> Connectors:bornier5
- P1: footprint (none) -> Potentiometers:Potentiometer_WirePads_Small
- Q1, Q2: footprint (none) -> TO_SOT_Packages_THT:TO-92_Inline_Narrow_Oval
- R1, R10, R11, R12, R13, R2, R3, R4, R5, R6, R7, R8, R9: footprint (none) -> Resistors_THT:R_Axial_DIN0411_L9.9mm_D3.6mm_P12.70mm_Horizontal
Connections:
- no-connect marks 23 -> 25

Commit message: 220930
Parts:
- removed J3: DB9M, Connectors:DB9MC, symbol DB9
- removed JP1, JP2: Jumper_NO_Small, Socket_Strips:Socket_Strip_Straight_1x02, symbol Jumper_NO_Small
- removed JP3, JP4: Jumper_NC_Small, Socket_Strips:Socket_Strip_Straight_1x02, symbol Jumper_NC_Small
- removed P1: 10k, Potentiometers:Potentiometer_WirePads_Small, symbol POT_TRIM
- added J3: Screw_Terminal_1x03, Connectors:bornier3, symbol Screw_Terminal_1x03
- added Q1: BC109, TO_SOT_Packages_THT:TO-18-3, symbol BC548
- added R2: 10k, Resistors_THT:R_Axial_DIN0411_L9.9mm_D3.6mm_P12.70mm_Horizontal, symbol R
- added R3: 1k, Resistors_THT:R_Axial_DIN0411_L9.9mm_D3.6mm_P12.70mm_Horizontal, symbol R
- renumbered JP5 to JP1, JP6 to JP2, JP7 to JP3, Q1 to Q2, Q2 to Q3, R7 to R10, R8 to R11, R10 to R12, R12 to R13, R6 to R14, R9 to R15, R2 to R4, R3 to R5, R4 to R6, R5 to R7, R13 to R8, R11 to R9
Connections:
- net BC is gone; now on net GND: J4.1, U2.18 (GND)
- net RXD is gone; now on net RXD-TTL: U2.2 (GPIO1)
- net TXD is gone; now on net TXD-TTL: U2.1 (GPIO0)
- net +5V: now also R8.1, R9.1, U1.15 (LED+); no longer R1.1, R8.2, R9.2
- net DB4: now also U2.14 (GPIO10); no longer U2.9 (GPIO6)
- net DB5: now also U2.15 (GPIO11); no longer U2.10 (GPIO7)
- net DB6: now also U2.16 (GPIO12); no longer U2.11 (GPIO8)
- net DB7: now also U2.17 (GPIO13); no longer U2.12 (GPIO9)
- net EN: now also U2.19 (GPIO14); no longer U2.14 (GPIO10)
- net GND: now also JP2.2, JP3.2, U2.13 (GND), U2.23 (GND), U2.28 (GND), U2.3 (GND), U2.42 (GND), U2.8 (GND), J3.3, Q1.3 (E), R2.2; no longer U1.16 (LED-)
- net RS: now also U2.20 (GPIO15); no longer U2.15 (GPIO11)
- net RXD-RS232C: now also J3.2
- net TXD-RS232C: now also J3.1
- net RXD1: now reaches Q3.1 (C), R5.2
- net RXD1: now also U2.12 (GPIO9)
- net TXD1: now reaches R6.1
- net TXD1: now also U2.11 (GPIO8)
- net at U2.24 (GPIO18): now also J4.2, R11.2
- net at U2.25 (GPIO19): now also J4.3, R10.2
- net at U2.26 (GPIO20): now also J4.4, R8.2
- net at U2.27 (GPIO21): now also J4.5, R9.2
- removed net -AS: JP2.2, R9.1, U2.22 (GPIO17)
- removed net -BD: J4.4, R11.2, U2.17 (GPIO13)
- removed net -BL: J4.3, R12.2, U2.19 (GPIO14)
- removed net -BR: J4.2, R13.2, U2.20 (GPIO15)
- removed net -BU: J4.5, R10.2, U2.16 (GPIO12)
- removed net -LB: JP3.2, R8.1, U2.21 (GPIO16)
- net -RST: no longer names the net of JP1.1, U2.30 (RUN)
- net BL+: no longer names the net of R1.2
- net BL+: now also Q1.1 (C); no longer U1.15 (LED+)
- net CONT: no longer names the net of U1.3 (Vo)
- net CONT: now also R2.1
- removed net JC: JP2.1, JP3.1, U2.23 (GND)
- new net: R1.1, U1.16 (LED-)
- new net: JP3.1, R13.2, U2.21 (GPIO16)
- new net: JP2.1, R12.2, U2.22 (GPIO17)
- new net: Q1.2 (B), R3.1
- new net BL: R3.2, U2.9 (GPIO6)
- no-connect marks 25 -> 11
Other:
- moved on the sheet: C1, C2, C3, C4, C5, D1, D2, F1, J1, J2, J4, JP1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

Commit message: 220930
Parts:
- removed J4: Screw_Terminal_1x05, Connectors:bornier5, symbol Screw_Terminal_1x05
- added J4: Screw_Terminal_1x07, Bornier:bornier7, symbol Screw_Terminal_1x07
- added R10, R11, R12, R13, R14, R15, R16, R9: 1k, Resistors_THT:R_Axial_DIN0309_L9.0mm_D3.2mm_P5.08mm_Vertical, symbol R
- added R24, R25: 10k, Resistors_THT:R_Axial_DIN0309_L9.0mm_D3.2mm_P5.08mm_Vertical, symbol R
- F1: value Fuse -> 1A F
- R1: renamed from R7; footprint Resistors_THT:R_Axial_DIN0411_L9.9mm_D3.6mm_P12.70mm_Horizontal -> Resistors_THT:R_Axial_DIN0309_L9.0mm_D3.2mm_P5.08mm_Vertical
- R17: renamed from R3; footprint Resistors_THT:R_Axial_DIN0411_L9.9mm_D3.6mm_P12.70mm_Horizontal -> Resistors_THT:R_Axial_DIN0309_L9.0mm_D3.2mm_P5.08mm_Vertical
- R18: renamed from R9; footprint Resistors_THT:R_Axial_DIN0411_L9.9mm_D3.6mm_P12.70mm_Horizontal -> Resistors_THT:R_Axial_DIN0309_L9.0mm_D3.2mm_P5.08mm_Vertical
- R19: renamed from R8; footprint Resistors_THT:R_Axial_DIN0411_L9.9mm_D3.6mm_P12.70mm_Horizontal -> Resistors_THT:R_Axial_DIN0309_L9.0mm_D3.2mm_P5.08mm_Vertical
- R2: renamed from R14; footprint Resistors_THT:R_Axial_DIN0411_L9.9mm_D3.6mm_P12.70mm_Horizontal -> Resistors_THT:R_Axial_DIN0309_L9.0mm_D3.2mm_P5.08mm_Vertical
- R20: renamed from R10; footprint Resistors_THT:R_Axial_DIN0411_L9.9mm_D3.6mm_P12.70mm_Horizontal -> Resistors_THT:R_Axial_DIN0309_L9.0mm_D3.2mm_P5.08mm_Vertical
- R21: renamed from R11; footprint Resistors_THT:R_Axial_DIN0411_L9.9mm_D3.6mm_P12.70mm_Horizontal -> Resistors_THT:R_Axial_DIN0309_L9.0mm_D3.2mm_P5.08mm_Vertical
- R22: renamed from R12; footprint Resistors_THT:R_Axial_DIN0411_L9.9mm_D3.6mm_P12.70mm_Horizontal -> Resistors_THT:R_Axial_DIN0309_L9.0mm_D3.2mm_P5.08mm_Vertical
- R23: renamed from R13; footprint Resistors_THT:R_Axial_DIN0411_L9.9mm_D3.6mm_P12.70mm_Horizontal -> Resistors_THT:R_Axial_DIN0309_L9.0mm_D3.2mm_P5.08mm_Vertical
- R3: renamed from R4; footprint Resistors_THT:R_Axial_DIN0411_L9.9mm_D3.6mm_P12.70mm_Horizontal -> Resistors_THT:R_Axial_DIN0309_L9.0mm_D3.2mm_P5.08mm_Vertical
- R4: renamed from R15; footprint Resistors_THT:R_Axial_DIN0411_L9.9mm_D3.6mm_P12.70mm_Horizontal -> Resistors_THT:R_Axial_DIN0309_L9.0mm_D3.2mm_P5.08mm_Vertical
- R5: renamed from R6; footprint Resistors_THT:R_Axial_DIN0411_L9.9mm_D3.6mm_P12.70mm_Horizontal -> Resistors_THT:R_Axial_DIN0309_L9.0mm_D3.2mm_P5.08mm_Vertical
- R6: renamed from R5; footprint Resistors_THT:R_Axial_DIN0411_L9.9mm_D3.6mm_P12.70mm_Horizontal -> Resistors_THT:R_Axial_DIN0309_L9.0mm_D3.2mm_P5.08mm_Vertical
- R7: renamed from R2; footprint Resistors_THT:R_Axial_DIN0411_L9.9mm_D3.6mm_P12.70mm_Horizontal -> Resistors_THT:R_Axial_DIN0309_L9.0mm_D3.2mm_P5.08mm_Vertical
- R8: renamed from R1; footprint Resistors_THT:R_Axial_DIN0411_L9.9mm_D3.6mm_P12.70mm_Horizontal -> Resistors_THT:R_Axial_DIN0309_L9.0mm_D3.2mm_P5.08mm_Vertical
- U2: value Pico -> Raspberry Pi Pico; footprint RPi_Pico:RPi_Pico_SMD_TH -> MCU_RaspberryPi_and_Boards:RPi_Pico_SMD_TH
- renumbered C5 to C3, C3 to C4, C4 to C5, Q2 to Q1, Q3 to Q2, Q1 to Q3
Connections:
- net +5V: now also R24.1, R25.1
- net BL: now also U2.19 (GPIO14); no longer U2.9 (GPIO6)
- net EN: now also U2.10 (GPIO7); no longer U2.19 (GPIO14)
- net GND: now also JP2.1, JP3.1, J4.1; no longer JP2.2, JP3.2
- net RS: now also U2.9 (GPIO6); no longer U2.20 (GPIO15)
- net at U2.24 (GPIO18): now also R13.2; no longer R21.2
- net at U2.25 (GPIO19): now also R12.2; no longer R20.2
- net at U2.26 (GPIO20): now also R11.2; no longer R19.2
- net at U2.27 (GPIO21): now also R10.2; no longer R18.2
- net at U2.29 (GPIO22): now also R9.2
- net RXD-RS232C renamed RXD1-RS232C
- net RXD-TTL renamed RXD0
- net TXD-RS232C renamed TXD1-RS232C
- net TXD-TTL renamed TXD0
- new net: R16.2, U2.20 (GPIO15)
- new net: R15.2, U2.21 (GPIO16)
- new net: R14.2, U2.22 (GPIO17)
- new net: JP3.2, R16.1, R25.2
- new net: JP2.2, R15.1, R24.2
- new net PB0: J4.2, R14.1, R23.2
- new net PB1: J4.3, R13.1, R22.2
- new net PB2: J4.4, R12.1, R21.2
- new net PB3: J4.5, R11.1, R20.2
- new net PB4: J4.6, R10.1, R19.2
- new net PB5: J4.7, R18.2, R9.1
- no-connect marks 11 -> 9
Other:
- moved on the sheet: C1, C2, C3, C4, C5, D1, D2, F1, J1, J2, J3, JP1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

Commit message: 221009
Connections:
- net +5V: now also U1.2 (VDD); no longer U1.1 (VSS)
- net GND: now also U1.1 (VSS); no longer U1.2 (VDD)
Changed lines of the file:
@@
 L GND #PWR07
 U 1 1 6335DEFB
-P 6200 2800
-F 0 "#PWR07" H 6200 2550 50  0001 C CNN
-F 1 "GND" H 6200 2650 50  0000 C CNN
-F 2 "" H 6200 2800 50  0000 C CNN
-F 3 "" H 6200 2800 50  0000 C CNN
-	1    6200 2800
+P 6100 2750
+F 0 "#PWR07" H 6100 2500 50  0001 C CNN
+F 1 "GND" H 6100 2600 50  0000 C CNN
+F 2 "" H 6100 2750 50  0000 C CNN
+F 3 "" H 6100 2750 50  0000 C CNN
+	1    6100 2750
 	1    0    0    -1
 $EndComp
@@
 U 1 1 6336E0EE
 P 6300 2200
-F 0 "R7" H 6100 2250 50  0000 C CNN
-F 1 "10k" H 6100 2150 50  0000 C CNN
+F 0 "R7" H 6200 2250 50  0000 C CNN
+F 1 "10k" H 6200 2050 50  0000 C CNN
 F 2 "Resistors_THT:R_Axial_DIN0309_L9.0mm_D3.2mm_P5.08mm_Vertical" V 6230 2200 50  0001 C CNN
 F 3 "" H 6300 2200 50  0000 C CNN
@@
 	5100 2950 2150 2950
 Wire Wire Line
-	6200 1800 6200 2800
-Wire Wire Line
 	6500 2650 6500 1800
-Wire Wire Line
-	6100 1900 6100 1800
 Wire Wire Line
 	7400 1800 7400 3200
@@
 	5800 1900 7500 1900
 Wire Wire Line
-	6200 2650 7600 2650
-Connection ~ 6200 2650
+	6100 2650 7600 2650
 Wire Wire Line
 	7600 2650 7600 2600
@@
 Wire Wire Line
 	7500 1900 7500 1800
-Connection ~ 6100 1900
 Wire Wire Line
 	5800 1800 5800 1900
@@
 Connection ~ 8750 3750
 Connection ~ 8850 3750
+Wire Wire Line
+	6200 1800 6200 1900
+Connection ~ 6200 1900
+Wire Wire Line
+	6100 1800 6100 2750
+Connection ~ 6100 2650
 $EndSCHEMATC

Commit message: 221018
Parts:
- JP2: Function Autoscroll -> Operation
- JP3: Function Line break -> modes
Connections:
- net GND: now also JP1.1; no longer JP1.2
- net at U2.30 (RUN): now also JP1.2; no longer JP1.1
Changed lines of the file:
@@
 U 1 1 63359C97
 P 7850 4600
-F 0 "JP1" H 7850 4675 50  0000 C CNN
+F 0 "JP1" H 7850 4500 50  0000 C CNN
 F 1 "Jumper_NO_Small" H 7860 4540 50  0001 C CNN
 F 2 "Socket_Strips:Socket_Strip_Straight_1x02" H 7850 4600 50  0001 C CNN
 F 3 "" H 7850 4600 50  0000 C CNN
-F 4 "Reset" H 7850 4525 60  0000 C CNN "Function"
+F 4 "Reset" H 7850 4700 60  0000 C CNN "Function"
 	1    7850 4600
-	0    -1   -1   0
+	0    1    1    0
 $EndComp
 Wire Wire Line
@@
 F 2 "Socket_Strips:Socket_Strip_Straight_1x02" H 8300 5950 50  0001 C CNN
 F 3 "" H 8300 5950 50  0000 C CNN
-F 4 "Line break" H 8300 6130 60  0000 C CNN "Function"
+F 4 "modes" H 8300 6130 60  0000 C CNN "Function"
 	1    8300 5950
 	1    0    0    1
@@
 F 2 "Socket_Strips:Socket_Strip_Straight_1x02" H 8300 5850 50  0001 C CNN
 F 3 "" H 8300 5850 50  0000 C CNN
-F 4 "Autoscroll" H 8300 5760 60  0000 C CNN "Function"
+F 4 "Operation" H 8300 5760 60  0000 C CNN "Function"
 	1    8300 5850
 	1    0    0    1
