File: cad_files/KiCAD/mini_serial_console.kicad_pcb (KiCad board)
At the start: 2 copper layers, 97.8 x 59.7 mm, 50 parts, among them J1 Screw_Terminal_1x02, J2 Screw_Terminal_1x03, J3 Screw_Terminal_1x03, J4 Screw_Terminal_1x07, Q1 BC559, Q2 BC548, Q3 BC109, U1 HD44780 compatible LCD, U2 Raspberry Pi Pico

Commit message: 221115
Connections:
- R18 pad 1: +5V -> Net-(R18-Pad1)
- R19 pad 1: +5V -> Net-(R18-Pad1)
- R20 pad 1: +5V -> Net-(R18-Pad1)
- R21 pad 1: +5V -> Net-(R18-Pad1)
- R22 pad 1: +5V -> Net-(R18-Pad1)
- R23 pad 1: +5V -> Net-(R18-Pad1)
- R24 pad 1: +5V -> Net-(R18-Pad1)
- R25 pad 1: +5V -> Net-(R18-Pad1)
- U2 pad 36: Net-(U2-Pad36) -> Net-(R18-Pad1)
Routing:
- net Net-(R18-Pad1): track 0.00 -> 150.5 mm
- net +5V: track 394.0 -> 331.1 mm

Commit message: 221201
Parts:
- F1: value 1A F -> 100mA F
Routing:
- net +5V: track 331.1 -> 369.9 mm
- net Net-(R18-Pad1): track 150.5 -> 111.8 mm
Changed lines of the file:
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@@
       (effects (font (size 1 1) (thickness 0.15)))
     )
-    (fp_text value "1A F" (at 0.635 5.715 180) (layer F.Fab)
+    (fp_text value "100mA F" (at 0.635 5.715 180) (layer F.Fab)
       (effects (font (size 1 1) (thickness 0.15)))
     )
@@
   (gr_line (start 96.012 128.524) (end 96.012 68.834) (angle 90) (layer Edge.Cuts) (width 0.15))
   (gr_line (start 193.802 128.524) (end 96.012 128.524) (angle 90) (layer Edge.Cuts) (width 0.15))
-  (segment (start 117.602 89.154) (end 119.126 89.154) (width 1) (layer F.Cu) (net 1) (status 400000))
-  (segment (start 121.92 80.264) (end 127.762 80.264) (width 1) (layer F.Cu) (net 1) (status 800000))
+  (segment (start 117.602 89.154) (end 119.126 89.154) (width 1) (layer F.Cu) (net 1))
+  (segment (start 121.92 80.264) (end 127.762 80.264) (width 1) (layer F.Cu) (net 1))
   (segment (start 120.396 81.788) (end 121.92 80.264) (width 1) (layer F.Cu) (net 1))
   (segment (start 120.396 87.884) (end 120.396 81.788) (width 1) (layer F.Cu) (net 1))
@@
   (segment (start 145.542 127.889) (end 147.447 127.889) (width 1) (layer F.Cu) (net 1))
   (segment (start 186.182 127.889) (end 186.817 127.254) (width 1) (layer F.Cu) (net 1))
+  (segment (start 147.447 127.889) (end 150.622 127.889) (width 1) (layer F.Cu) (net 1))
+  (segment (start 150.622 127.889) (end 154.432 127.889) (width 1) (layer F.Cu) (net 1))
+  (segment (start 154.432 127.889) (end 158.242 127.889) (width 1) (layer F.Cu) (net 1))
+  (segment (start 158.242 127.889) (end 162.052 127.889) (width 1) (layer F.Cu) (net 1))
+  (segment (start 162.052 127.889) (end 165.862 127.889) (width 1) (layer F.Cu) (net 1))
+  (segment (start 165.862 127.889) (end 186.182 127.889) (width 1) (layer F.Cu) (net 1))
   (segment (start 185.594 76.454) (end 185.594 80.217) (width 1) (layer F.Cu) (net 2))
   (segment (start 185.594 80.217) (end 185.547 80.264) (width 1) (layer F.Cu) (net 2))
@@
   (segment (start 146.177 88.519) (end 146.812 89.154) (width 0.25) (layer F.Cu) (net 52))
   (segment (start 144.907 88.519) (end 146.177 88.519) (width 0.25) (layer F.Cu) (net 52))
-  (segment (start 122.682 89.154) (end 125.476 91.948) (width 1) (layer F.Cu) (net 53) (status 400000))
-  (segment (start 142.748 121.285) (end 145.542 124.079) (width 1) (layer F.Cu) (net 53) (status 800000))
+  (segment (start 122.682 89.154) (end 125.476 91.948) (width 1) (layer F.Cu) (net 53))
+  (segment (start 142.748 121.285) (end 145.542 124.079) (width 1) (layer F.Cu) (net 53))
   (segment (start 142.748 110.744) (end 142.748 121.285) (width 1) (layer F.Cu) (net 53))
   (segment (start 141.224 109.22) (end 142.748 110.744) (width 1) (layer F.Cu) (net 53))
@@
   (segment (start 125.476 101.6) (end 125.476 106.68) (width 1) (layer F.Cu) (net 53))
   (segment (start 125.476 91.948) (end 125.476 101.6) (width 1) (layer F.Cu) (net 53))
-  (segment (start 181.102 103.124) (end 181.102 122.936) (width 1) (layer B.Cu) (net 53) (status 400000))
+  (segment (start 181.102 103.124) (end 181.102 122.936) (width 1) (layer B.Cu) (net 53))
   (segment (start 181.102 122.936) (end 179.959 124.079) (width 1) (layer B.Cu) (net 53))
-  (segment (start 179.959 124.079) (end 145.542 124.079) (width 1) (layer B.Cu) (net 53) (status 800000))
-  (segment (start 147.447 127.889) (end 150.622 127.889) (width 1) (layer F.Cu) (net 53))
-  (segment (start 150.622 127.889) (end 154.432 127.889) (width 1) (layer F.Cu) (net 53))
-  (segment (start 154.432 127.889) (end 158.242 127.889) (width 1) (layer F.Cu) (net 53))
-  (segment (start 158.242 127.889) (end 162.052 127.889) (width 1) (layer F.Cu) (net 53))
-  (segment (start 162.052 127.889) (end 165.862 127.889) (width 1) (layer F.Cu) (net 53))
-  (segment (start 165.862 127.889) (end 186.182 127.889) (width 1) (layer F.Cu) (net 53))
+  (segment (start 179.959 124.079) (end 145.542 124.079) (width 1) (layer B.Cu) (net 53))
   (segment (start 122.682 85.344) (end 122.682 89.154) (width 1) (layer F.Cu) (net 53))
 )
